Commit message: Add files via upload

File: joints_act/urdf/fixed_ex.urdf (robot description, URDF)
Before this commit: robot link_example, 7 links, 6 joints
Links:
- link base_link: geometry visual mesh filename=package://puzzlebot_sim/meshes/Puzzlebot_Jetson_Lidar_Editi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
- link caster_link: geometry visual mesh filename=package://puzzlebot_sim/meshes/Puzzlebot_Caster_Wheel.stl
- link wheel_l_link: geometry visual mesh filename=package://puzzlebot_sim/meshes/Puzzlebot_Wheel.stl
- link wheel_r_link: geometry visual mesh filename=package://puzzlebot_sim/meshes/Puzzlebot_Wheel.stl
Joints:
- joint wheel_l_joint: axis 1 0 0 -> 0 1 0
- joint wheel_r_joint: axis 1 0 0 -> 0 1 0
